File: junon-kb.kicad_pcb (KiCad board)
At the start: 2 copper layers, 133 x 95 mm, 61 parts, among them IC1 BD41041FJ-CE2, J1 STLINK-V3MINIE, J2 SJ-43514-SMT-TR, J3 SJ-43514-SMT-TR, J4 632723300011, U1 STM32G473CCT3, U3 SPX3819M5-L-1-5/TR, Y1 ECS-3225MV-320-CN-TR

Commit message: update NRST
Connections:
- C1 pad 1: Net-(U1A-PG10-NRST) -> /MCU/NRST
- J1 pad 9: GND -> /MCU/NRST
- RST1 pad 1: Net-(U1A-PG10-NRST) -> /MCU/NRST
- U1 pad 7: Net-(U1A-PG10-NRST) -> /MCU/NRST
Routing:
- net /MCU/NRST: track 0.00 -> 50.0 mm, vias 0 -> 2
- net Net-(U1A-PG10-NRST): track 31.5 -> 0.00 mm, vias 2 -> 0
- net +3V3: track 27.3 -> 30.7 mm, vias 7 -> 9
- net GND: track 96.5 -> 98.3 mm
- net /MCU/S6: track 105.7 -> 104.8 mm
- net /MCU/ROTARY_SW: track 14.2 -> 15.0 mm

Commit message: flesh out SWD circuit
Parts:
- added R4: 22R, Resistor_SMD:R_01005_0402Metric, F.Cu at (195.2, 94.0)
- added R5: 10K, junon-kb:RES_RK73H1E_KOA, F.Cu at (195.7, 91.6)
- added R6: 10K, junon-kb:RES_RK73H1E_KOA, F.Cu at (195.2, 95.8)
- added R7: 10K, junon-kb:RES_RK73H1E_KOA, F.Cu at (191.8, 69.8)
Connections:
- D1 pad 5: unconnected-(D1-VBUS-Pad5) -> /USB/VBUS
- J1 pad 3: /MCU/SWD_IO -> Net-(J1-JTMS/SWDIO)
Routing:
- net GND: track 98.3 -> 104.5 mm, vias 12 -> 13
- net Net-(J1-JTMS/SWDIO): track 0.00 -> 4.83 mm
- net +3V3: track 30.7 -> 33.2 mm, vias 9 -> 11
- net /USB/VBUS: track 18.2 -> 20.5 mm, vias 1 -> 2
- net /MCU/NRST: track 50.0 -> 52.0 mm, vias 2 -> 3
- net /MCU/SWD_CLK: track 4.06 -> 4.94 mm

Commit message: next version
Routing:
- net GND: track 104.5 -> 103.0 mm
