File: MCU.kicad_sch (KiCad schematic)
At the start: 14 parts, among them U1 STM32G473CCT3, Y1 ECS-3225MV-320-CN-TR

Commit message: update NRST
Connections:
- net NRST: now reaches C1.1, RST1.1, U1.7 (PG10-NRST)
Changed lines of the file:
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@@
   (junction (at 210.82 48.26) (diameter 0) (color 0 0 0 0)
   )
+  (junction (at 132.08 77.47) (diameter 0) (color 0 0 0 0)
+  )
   (junction (at 210.82 58.42) (diameter 0) (color 0 0 0 0)
   )
@@
     (stroke (width 0) (type default))
   )
+  (wire (pts (xy 132.08 77.47) (xy 132.08 89.408))
+    (stroke (width 0) (type default))
+  )
   (wire (pts (xy 243.205 104.14) (xy 246.38 104.14))
     (stroke (width 0) (type default))
@@
   )
   (wire (pts (xy 196.85 63.5) (xy 194.31 63.5))
+    (stroke (width 0) (type default))
+  )
+  (wire (pts (xy 132.08 89.408) (xy 136.906 89.408))
     (stroke (width 0) (type default))
   )
@@
     (effects (font (size 1.27 1.27)) (justify right))
   )
+  (hierarchical_label "NRST" (shape input) (at 136.906 89.408 0) (fields_autoplaced)
+    (effects (font (size 1.27 1.27)) (justify left))
+  )
   (hierarchical_label "SWD_CLK" (shape input) (at 52.705 88.9 180) (fields_autoplaced)
