File: usb.kicad_sch (KiCad schematic)
At the start: 7 parts, among them J4 632723300011

Commit message: flesh out SWD circuit
Connections:
- net VBUS: now also D1.5 (VBUS)
Changed lines of the file:
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@@
+    (stroke (width 0) (type default))
+  )
+  (wire (pts (xy 207.645 78.105) (xy 212.852 78.105))
     (stroke (width 0) (type default))
   )
@@
     (effects (font (size 1.27 1.27)) (justify right bottom))
   )
+  (label "VBUS" (at 212.852 78.105 180) (fields_autoplaced)
+    (effects (font (size 1.27 1.27)) (justify right bottom))
+  )
